Commit message: Add files via upload

File: ros_odrive/my_odrive_botwheel_explorer/description/urdf/diffbot_description.urdf.xacro (robot description, xacro)
@@ -5,13 +5,23 @@
   <xacro:property name="PI" value="3.1415926535897931"/>
   <xacro:property name="base_mass" value="0.3" /> <!-- arbitrary value for base mass -->
-  <xacro:property name="base_width" value="0.1" />
-  <xacro:property name="base_length" value="0.1" />
+  <xacro:property name="base_width" value="0.4" />
+  <xacro:property name="base_length" value="0.3" />
   <xacro:property name="base_height" value="0.05" />
   <xacro:property name="wheel_mass" value="0.3" /> <!-- arbitrary value for wheel mass -->
   <xacro:property name="wheel_len" value="0.020" />
   <xacro:property name="wheel_radius" value="0.015" />
-  <xacro:property name="caster_wheel_mass" value="0.1" /> <!-- arbitrary value for caster wheel mass -->
-  <xacro:property name="caster_wheel_radius" value="0.015" />
   <xacro:property name="z_offset" value="-${base_height/2}" /> <!-- Space btw top of beam and the each joint -->
+  <material name="white">
+      <color rgba="1 1 1 1" />
+  </material>
+  <material name="orange">
+      <color rgba="1 0.3 0.1 1"/>
+  </material>
+  <material name="blue">
+      <color rgba="0.2 0.2 1 1"/>
+  </material>
+  <material name="black">
+      <color rgba="0 0 0 1"/>
+  </material>
   <!-- Base Link -->
   <link name="${prefix}base_link">
